File: Sydney/Sydney.kicad_sch (KiCad schematic)
At the start: 0 parts

Commit message: commit stuff
Parts:
- added C1: C, Capacitor_SMD:C_0603_1608Metric_Pad1.08x0.95mm_HandSolder, symbol Device:C
- added D1: LED, LED_SMD:LED_0805_2012Metric_Pad1.15x1.40mm_HandSolder, symbol Device:LED
- added J1: Conn_01x02_Pin, Taranium-libs:25x_48mm NFC Antenna, symbol Connector:Conn_01x02_Pin
- added R1: R, Resistor_SMD:R_0603_1608Metric_Pad0.98x0.95mm_HandSolder, symbol Device:R
- added U1: NT3H2111W0FHKH, Taranium-libs:QFN8P50_160X160X50L40X20N, symbol Taranium-libs:NT3H2111W0FHKH
Connections:
- new net: C1.1, R1.1, U1.6 (VCC), U1.7 (VOUT)
- new net: C1.2, D1.1 (K), U1.2 (VSS)
- new net: J1.1 (Pin_1), U1.8 (LB)
- new net: J1.2 (Pin_2), U1.1 (LA)
- new net: D1.2 (A), R1.2
