File: Brisbane/Organiser/Sydney.kicad_pcb (KiCad board)
At the start: 2 copper layers, 99.1 x 54 mm, 6 parts, among them J1 Conn_01x02_Pin, U1 NT3H2111W0FHKH

Commit message: potato
Parts:
- removed C1: C, Capacitor_SMD:C_0603_1608Metric_Pad1.08x0.95mm_HandSolder
- removed D1: LED, LED_SMD:LED_0805_2012Metric_Pad1.15x1.40mm_HandSolder
- removed J1: Conn_01x02_Pin, Taranium-libs:25x_48mm NFC Antenna
- removed R1: R, Resistor_SMD:R_0603_1608Metric_Pad0.98x0.95mm_HandSolder
- removed U1: NT3H2111W0FHKH, Taranium-libs:QFN8P50_160X160X50L40X20N
Routing:
- net Net-(J1-Pin_1): track 47.5 -> 0.00 mm
- net Net-(J1-Pin_2): track 42.6 -> 0.00 mm, vias 2 -> 0
- net Net-(D1-K): track 9.60 -> 0.00 mm
- net Net-(U1-VCC): track 6.13 -> 0.00 mm
- net Net-(D1-A): track 2.53 -> 0.00 mm
